File: IRSensorArray.sch (KiCad schematic (older format))
At the start: 27 parts

Commit message: Connected jumpers and ADC
Parts:
- added J?: PASSTHRU, symbol Connector:Conn_01x04_Female
- added J?: EXT_REF, symbol Connector:Conn_01x01_Female
- C?: value C -> 100nF
- C?: value CP -> 1uF
- C?: value CP -> 10uF
- C?: value CP -> 0.1uF
- J?: value Conn_01x04_Female -> INPUT
- R? (x2): value R -> 10k0
Connections:
- net labels added: CH0, CH1, CH2, CH3, CH4, CH5, CH6, CH7, REF, SB_0, SB_1
- wire segments 0 -> 34
Other:
- note added: "ADC"
- note added: "Reference Voltage Select"
- note added: "Slave Address Select"
- note added: "To use 5V bus as reference, connect center to pin 1\nTo use internal 2.5V reference, leave disconnected\nTo use external 5V reference, connect center to 3 \nand connect EXT_REF to 5V precision reference"

Commit message: Added sensor array
Parts:
- removed D? (x8): LED, symbol Device:LED
- removed R? (x8): R, symbol Device:R
Connections:
- net labels added: SCL, SDA
- wire segments 34 -> 70
Other:
- note added: "IR Array"
- note added: "Power Input"
- note added: "Todo: make it so \nyou can't short this"
- note added: "Todo:\nCalculate pullups\nfor I2C speeds"
