File: IRSensorArray.sch (KiCad schematic (older format))
At the start: 13 parts, among them J1 EXT_REF, J2 INPUT, J3 PASSTHRU, U1 ADS7828

Commit message: Changed triangle solder bridges to semi-circle
Parts:
- JP1, JP2, JP3: footprint footprints:SolderJumper-3_P2.0mm_Open_TrianglePad1.0x1.5mm -> footprints:SolderJumper-3_P1.3mm_Open_RoundedPad1.0x1.5mm_NumberLabels
Changed lines of the file:
@@
 F 0 "JP1" V 3000 2200 50  0000 C CNN
 F 1 "SB_0" V 2900 2200 50  0000 C CNN
-F 2 "footprints:SolderJumper-3_P2.0mm_Open_TrianglePad1.0x1.5mm" H 2950 2000 50  0001 C CNN
+F 2 "footprints:SolderJumper-3_P1.3mm_Open_RoundedPad1.0x1.5mm_NumberLabels" H 2950 2000 50  0001 C CNN
 F 3 "~" H 2950 2000 50  0001 C CNN
 	1    2950 2000
@@
 F 0 "JP3" V 3850 2200 50  0000 C CNN
 F 1 "SB_1" V 3750 2200 50  0000 C CNN
-F 2 "footprints:SolderJumper-3_P2.0mm_Open_TrianglePad1.0x1.5mm" H 3800 2000 50  0001 C CNN
+F 2 "footprints:SolderJumper-3_P1.3mm_Open_RoundedPad1.0x1.5mm_NumberLabels" H 3800 2000 50  0001 C CNN
 F 3 "~" H 3800 2000 50  0001 C CNN
 	1    3800 2000
@@
 F 0 "JP2" V 3500 4000 50  0000 C CNN
 F 1 "REF_5V" V 3400 4000 50  0000 C CNN
-F 2 "footprints:SolderJumper-3_P2.0mm_Open_TrianglePad1.0x1.5mm" H 3450 3750 50  0001 C CNN
+F 2 "footprints:SolderJumper-3_P1.3mm_Open_RoundedPad1.0x1.5mm_NumberLabels" H 3450 3750 50  0001 C CNN
 F 3 "~" H 3450 3750 50  0001 C CNN
 	1    3450 3750

Commit message: First draft finished!
Parts:
- removed C3: 1uF, Capacitors_THT:CP_Radial_D4.0mm_P2.00mm, symbol Device:CP
Connections:
- wire segments 70 -> 66
Changed lines of the file:
@@
 L Device:C C4
 U 1 1 5B22D6A1
-P 8700 3250
-F 0 "C4" H 8815 3296 50  0000 L CNN
-F 1 "100nF" H 8815 3205 50  0000 L CNN
-F 2 "Capacitors_THT:C_Disc_D5.1mm_W3.2mm_P5.00mm" H 8738 3100 50  0001 C CNN
-F 3 "~" H 8700 3250 50  0001 C CNN
-	1    8700 3250
-	1    0    0    -1
-$EndComp
-$Comp
-L Device:CP C3
-U 1 1 5B22D7EA
-P 8250 3250
-F 0 "C3" H 8368 3296 50  0000 L CNN
-F 1 "1uF" H 8368 3205 50  0000 L CNN
-F 2 "Capacitors_THT:CP_Radial_D4.0mm_P2.00mm" H 8288 3100 50  0001 C CNN
-F 3 "~" H 8250 3250 50  0001 C CNN
-	1    8250 3250
+P 8500 3250
+F 0 "C4" H 8615 3296 50  0000 L CNN
+F 1 "100nF" H 8615 3205 50  0000 L CNN
+F 2 "Capacitors_THT:C_Disc_D5.1mm_W3.2mm_P5.00mm" H 8538 3100 50  0001 C CNN
+F 3 "~" H 8500 3250 50  0001 C CNN
+	1    8500 3250
 	1    0    0    -1
 $EndComp
@@
 L Device:CP C2
 U 1 1 5B22D97A
-P 7800 3250
-F 0 "C2" H 7918 3296 50  0000 L CNN
-F 1 "10uF" H 7918 3205 50  0000 L CNN
-F 2 "Capacitors_THT:CP_Radial_D5.0mm_P2.00mm" H 7838 3100 50  0001 C CNN
-F 3 "~" H 7800 3250 50  0001 C CNN
-	1    7800 3250
+P 7950 3250
+F 0 "C2" H 8068 3296 50  0000 L CNN
+F 1 "10uF" H 8068 3205 50  0000 L CNN
+F 2 "Capacitors_THT:CP_Radial_D5.0mm_P2.00mm" H 7988 3100 50  0001 C CNN
+F 3 "~" H 7950 3250 50  0001 C CNN
+	1    7950 3250
 	1    0    0    -1
 $EndComp
@@
 	8700 2000 8700 1850
 Wire Wire Line
+	8800 2100 8300 2100
+Wire Wire Line
 	8800 2200 8300 2200
-Wire Wire Line
-	8800 2100 8300 2100
+Text Label 8300 2200 0    50   ~ 0
+SDA
 Text Label 8300 2100 0    50   ~ 0
-SDA
-Text Label 8300 2200 0    50   ~ 0
 SCL
 $Comp
@@
 	7700 2000 7700 1850
 Wire Wire Line
+	7800 2100 7300 2100
+Wire Wire Line
 	7800 2200 7300 2200
-Wire Wire Line
-	7800 2100 7300 2100
+Text Label 7300 2200 0    50   ~ 0
+SDA
 Text Label 7300 2100 0    50   ~ 0
-SDA
-Text Label 7300 2200 0    50   ~ 0
 SCL
 $Comp
 L power:GND #PWR0116
 U 1 1 5B29CE6A
-P 8450 3550
-F 0 "#PWR0116" H 8450 3300 50  0001 C CNN
-F 1 "GND" H 8455 3377 50  0000 C CNN
-F 2 "" H 8450 3550 50  0001 C CNN
-F 3 "" H 8450 3550 50  0001 C CNN
-	1    8450 3550
+P 8250 3550
+F 0 "#PWR0116" H 8250 3300 50  0001 C CNN
+F 1 "GND" H 8255 3377 50  0000 C CNN
+F 2 "" H 8250 3550 50  0001 C CNN
+F 3 "" H 8250 3550 50  0001 C CNN
+	1    8250 3550
 	1    0    0    -1
 $EndComp
@@
 L power:+5V #PWR0117
 U 1 1 5B29CEAF
-P 8450 2950
-F 0 "#PWR0117" H 8450 2800 50  0001 C CNN
-F 1 "+5V" H 8465 3123 50  0000 C CNN
-F 2 "" H 8450 2950 50  0001 C CNN
-F 3 "" H 8450 2950 50  0001 C CNN
-	1    8450 2950
-	1    0    0    -1
-$EndComp
-Wire Wire Line
-	8700 3100 8700 3050
-Wire Wire Line
-	8700 3050 8450 3050
-Wire Wire Line
-	7800 3050 7800 3100
-Wire Wire Line
-	8250 3100 8250 3050
+P 8250 2950
+F 0 "#PWR0117" H 8250 2800 50  0001 C CNN
+F 1 "+5V" H 8265 3123 50  0000 C CNN
+F 2 "" H 8250 2950 50  0001 C CNN
+F 3 "" H 8250 2950 50  0001 C CNN
+	1    8250 2950
+	1    0    0    -1
+$EndComp
+Wire Wire Line
+	8500 3100 8500 3050
+Wire Wire Line
+	8500 3050 8250 3050
+Wire Wire Line
+	7950 3050 7950 3100
+Wire Wire Line
+	8250 2950 8250 3050
 Connection ~ 8250 3050
 Wire Wire Line
-	8250 3050 7800 3050
-Wire Wire Line
-	8450 2950 8450 3050
-Connection ~ 8450 3050
-Wire Wire Line
-	8450 3050 8250 3050
-Wire Wire Line
-	7800 3400 7800 3450
-Wire Wire Line
-	7800 3450 8250 3450
-Wire Wire Line
-	8700 3450 8700 3400
-Wire Wire Line
-	8250 3450 8250 3400
+	7950 3400 7950 3450
+Wire Wire Line
+	8500 3450 8500 3400
+Wire Wire Line
+	8250 3550 8250 3450
 Connection ~ 8250 3450
 Wire Wire Line
-	8250 3450 8450 3450
-Wire Wire Line
-	8450 3550 8450 3450
-Connection ~ 8450 3450
-Wire Wire Line
-	8450 3450 8700 3450
+	8250 3450 8500 3450
 Wire Notes Line
 	7050 3950 9550 3950
@@
 Wire Notes Line
 	4450 5650 9550 5650
+Wire Wire Line
+	7950 3050 8250 3050
+Wire Wire Line
+	7950 3450 8250 3450
 $EndSCHEMATC

Commit message: Added images
Parts:
- R1, R2: DNP (none) -> DNP
Other:
- note removed: "Todo: make it so \nyou can't short this"
- note removed: "Todo:\nCalculate pullups\nfor I2C speeds"

Commit message: Added reverse voltage diode
Parts:
- added D?: 1N4007, symbol Device:D
Connections:
- net labels added: VCC
- wire segments 66 -> 69
Changed lines of the file:
@@
 L Device:C C4
 U 1 1 5B22D6A1
-P 8400 3450
-F 0 "C4" H 8515 3496 50  0000 L CNN
-F 1 "100nF" H 8515 3405 50  0000 L CNN
-F 2 "Capacitors_THT:C_Disc_D5.1mm_W3.2mm_P5.00mm" H 8438 3300 50  0001 C CNN
-F 3 "~" H 8400 3450 50  0001 C CNN
-	1    8400 3450
+P 8750 3500
+F 0 "C4" H 8865 3546 50  0000 L CNN
+F 1 "100nF" H 8865 3455 50  0000 L CNN
+F 2 "Capacitors_THT:C_Disc_D5.1mm_W3.2mm_P5.00mm" H 8788 3350 50  0001 C CNN
+F 3 "~" H 8750 3500 50  0001 C CNN
+	1    8750 3500
 	1    0    0    -1
 $EndComp
@@
 L Device:CP C2
 U 1 1 5B22D97A
-P 7850 3450
-F 0 "C2" H 7968 3496 50  0000 L CNN
-F 1 "10uF" H 7968 3405 50  0000 L CNN
-F 2 "Capacitors_THT:CP_Radial_D5.0mm_P2.00mm" H 7888 3300 50  0001 C CNN
-F 3 "~" H 7850 3450 50  0001 C CNN
-	1    7850 3450
+P 8200 3500
+F 0 "C2" H 8318 3546 50  0000 L CNN
+F 1 "10uF" H 8318 3455 50  0000 L CNN
+F 2 "Capacitors_THT:CP_Radial_D5.0mm_P2.00mm" H 8238 3350 50  0001 C CNN
+F 3 "~" H 8200 3500 50  0001 C CNN
+	1    8200 3500
 	1    0    0    -1
 $EndComp
@@
 $EndComp
 $Comp
-L power:+5V #PWR0102
-U 1 1 5B22DDA3
-P 8600 2050
-F 0 "#PWR0102" H 8600 1900 50  0001 C CNN
-F 1 "+5V" H 8615 2223 50  0000 C CNN
-F 2 "" H 8600 2050 50  0001 C CNN
-F 3 "" H 8600 2050 50  0001 C CNN
-	1    8600 2050
-	1    0    0    -1
-$EndComp
-$Comp
 L power:+5V #PWR0103
 U 1 1 5B22E2FB
@@
 L power:+5V #PWR0110
 U 1 1 5B22F119
-P 5450 2050
-F 0 "#PWR0110" H 5450 1900 50  0001 C CNN
-F 1 "+5V" H 5465 2223 50  0000 C CNN
-F 2 "" H 5450 2050 50  0001 C CNN
-F 3 "" H 5450 2050 50  0001 C CNN
-	1    5450 2050
+P 5450 1850
+F 0 "#PWR0110" H 5450 1700 50  0001 C CNN
+F 1 "+5V" H 5465 2023 50  0000 C CNN
+F 2 "" H 5450 1850 50  0001 C CNN
+F 3 "" H 5450 1850 50  0001 C CNN
+	1    5450 1850
 	1    0    0    -1
 $EndComp
@@
 $EndComp
 Wire Wire Line
-	5450 2150 5450 2050
-Wire Wire Line
 	5450 3800 5450 3650
 Wire Wire Line
@@
 	1    0    0    -1
 $EndComp
-$Comp
-L power:+5V #PWR0115
-U 1 1 5B29A63D
-P 7600 2050
-F 0 "#PWR0115" H 7600 1900 50  0001 C CNN
-F 1 "+5V" H 7615 2223 50  0000 C CNN
-F 2 "" H 7600 2050 50  0001 C CNN
-F 3 "" H 7600 2050 50  0001 C CNN
-	1    7600 2050
-	1    0    0    -1
-$EndComp
 Wire Wire Line
 	7700 2200 7600 2200
@@
 L power:GND #PWR0116
 U 1 1 5B29CE6A
-P 8150 3750
-F 0 "#PWR0116" H 8150 3500 50  0001 C CNN
-F 1 "GND" H 8155 3577 50  0000 C CNN
-F 2 "" H 8150 3750 50  0001 C CNN
-F 3 "" H 8150 3750 50  0001 C CNN
-	1    8150 3750
+P 8500 3800
+F 0 "#PWR0116" H 8500 3550 50  0001 C CNN
+F 1 "GND" H 8505 3627 50  0000 C CNN
+F 2 "" H 8500 3800 50  0001 C CNN
+F 3 "" H 8500 3800 50  0001 C CNN
+	1    8500 3800
 	1    0    0    -1
 $EndComp
@@
 L power:+5V #PWR0117
 U 1 1 5B29CEAF
-P 8150 3150
-F 0 "#PWR0117" H 8150 3000 50  0001 C CNN
-F 1 "+5V" H 8165 3323 50  0000 C CNN
-F 2 "" H 8150 3150 50  0001 C CNN
-F 3 "" H 8150 3150 50  0001 C CNN
-	1    8150 3150
-	1    0    0    -1
-$EndComp
-Wire Wire Line
-	8400 3300 8400 3250
-Wire Wire Line
-	8400 3250 8150 3250
-Wire Wire Line
-	7850 3250 7850 3300
-Wire Wire Line
-	8150 3150 8150 3250
-Connection ~ 8150 3250
-Wire Wire Line
-	7850 3600 7850 3650
-Wire Wire Line
-	8400 3650 8400 3600
-Wire Wire Line
-	8150 3750 8150 3650
-Connection ~ 8150 3650
-Wire Wire Line
-	8150 3650 8400 3650
+P 8500 3200
+F 0 "#PWR0117" H 8500 3050 50  0001 C CNN
+F 1 "+5V" H 8515 3373 50  0000 C CNN
+F 2 "" H 8500 3200 50  0001 C CNN
+F 3 "" H 8500 3200 50  0001 C CNN
+	1    8500 3200
+	1    0    0    -1
+$EndComp
+Wire Wire Line
+	8750 3350 8750 3300
+Wire Wire Line
+	8750 3300 8500 3300
+Wire Wire Line
+	8200 3300 8200 3350
+Wire Wire Line
+	8500 3200 8500 3300
+Connection ~ 8500 3300
+Wire Wire Line
+	8200 3650 8200 3700
+Wire Wire Line
+	8750 3700 8750 3650
+Wire Wire Line
+	8500 3800 8500 3700
+Connection ~ 8500 3700
+Wire Wire Line
+	8500 3700 8750 3700
 Wire Notes Line
 	6950 4150 9450 4150
@@
 	4350 5850 9450 5850
 Wire Wire Line
-	7850 3250 8150 3250
-Wire Wire Line
-	7850 3650 8150 3650
+	8200 3300 8500 3300
+Wire Wire Line
+	8200 3700 8500 3700
+$Comp
+L Device:D D?
+U 1 1 5B2AEBA3
+P 7900 3300
+F 0 "D?" H 7900 3084 50  0000 C CNN
+F 1 "1N4007" H 7900 3175 50  0000 C CNN
+F 2 "" H 7900 3300 50  0001 C CNN
+F 3 "~" H 7900 3300 50  0001 C CNN
+	1    7900 3300
+	-1   0    0    1
+$EndComp
+Wire Wire Line
+	5450 1850 5450 2150
+$Comp
+L power:VCC #PWR?
+U 1 1 5B2AA17D
+P 7600 2050
+F 0 "#PWR?" H 7600 1900 50  0001 C CNN
+F 1 "VCC" H 7617 2223 50  0000 C CNN
+F 2 "" H 7600 2050 50  0001 C CNN
+F 3 "" H 7600 2050 50  0001 C CNN
+	1    7600 2050
+	1    0    0    -1
+$EndComp
+$Comp
+L power:VCC #PWR?
+U 1 1 5B2AA1A9
+P 8600 2050
+F 0 "#PWR?" H 8600 1900 50  0001 C CNN
+F 1 "VCC" H 8617 2223 50  0000 C CNN
+F 2 "" H 8600 2050 50  0001 C CNN
+F 3 "" H 8600 2050 50  0001 C CNN
+	1    8600 2050
+	1    0    0    -1
+$EndComp
+$Comp
+L power:VCC #PWR?
+U 1 1 5B2AA1CE
+P 7550 3200
+F 0 "#PWR?" H 7550 3050 50  0001 C CNN
+F 1 "VCC" H 7567 3373 50  0000 C CNN
+F 2 "" H 7550 3200 50  0001 C CNN
+F 3 "" H 7550 3200 50  0001 C CNN
+	1    7550 3200
+	1    0    0    -1
+$EndComp
+Wire Wire Line
+	7750 3300 7550 3300
+Wire Wire Line
+	7550 3300 7550 3200
+Wire Wire Line
+	8050 3300 8200 3300
+Connection ~ 8200 3300
 $EndSCHEMATC
