File: _saved_IRSensorArray.sch (KiCad schematic (older format))
At the start: 13 parts, among them J1 EXT_REF, J2 INPUT, J3 PASSTHRU, U1 ADS7828

Commit message: Added reverse voltage diode
Parts:
- D9: renamed from D?; footprint (none) -> Diodes_THT:D_DO-41_SOD81_P2.54mm_Vertical_AnodeUp
Connections:
- net labels added: VCC
Changed lines of the file:
@@
 L Device:C C4
 U 1 1 5B22D6A1
-P 8400 3450
-F 0 "C4" H 8515 3496 50  0000 L CNN
-F 1 "100nF" H 8515 3405 50  0000 L CNN
-F 2 "Capacitors_THT:C_Disc_D5.1mm_W3.2mm_P5.00mm" H 8438 3300 50  0001 C CNN
-F 3 "~" H 8400 3450 50  0001 C CNN
-	1    8400 3450
+P 8750 3500
+F 0 "C4" H 8865 3546 50  0000 L CNN
+F 1 "100nF" H 8865 3455 50  0000 L CNN
+F 2 "Capacitors_THT:C_Disc_D5.1mm_W3.2mm_P5.00mm" H 8788 3350 50  0001 C CNN
+F 3 "~" H 8750 3500 50  0001 C CNN
+	1    8750 3500
 	1    0    0    -1
 $EndComp
@@
 L Device:CP C2
 U 1 1 5B22D97A
-P 7850 3450
-F 0 "C2" H 7968 3496 50  0000 L CNN
-F 1 "10uF" H 7968 3405 50  0000 L CNN
-F 2 "Capacitors_THT:CP_Radial_D5.0mm_P2.00mm" H 7888 3300 50  0001 C CNN
-F 3 "~" H 7850 3450 50  0001 C CNN
-	1    7850 3450
+P 8200 3500
+F 0 "C2" H 8318 3546 50  0000 L CNN
+F 1 "10uF" H 8318 3455 50  0000 L CNN
+F 2 "Capacitors_THT:CP_Radial_D5.0mm_P2.00mm" H 8238 3350 50  0001 C CNN
+F 3 "~" H 8200 3500 50  0001 C CNN
+	1    8200 3500
 	1    0    0    -1
 $EndComp
@@
 $EndComp
 $Comp
-L power:+5V #PWR0102
-U 1 1 5B22DDA3
-P 8600 2050
-F 0 "#PWR0102" H 8600 1900 50  0001 C CNN
-F 1 "+5V" H 8615 2223 50  0000 C CNN
-F 2 "" H 8600 2050 50  0001 C CNN
-F 3 "" H 8600 2050 50  0001 C CNN
-	1    8600 2050
-	1    0    0    -1
-$EndComp
-$Comp
 L power:+5V #PWR0103
 U 1 1 5B22E2FB
@@
 L power:+5V #PWR0110
 U 1 1 5B22F119
-P 4900 1800
-F 0 "#PWR0110" H 4900 1650 50  0001 C CNN
-F 1 "+5V" H 4915 1973 50  0000 C CNN
-F 2 "" H 4900 1800 50  0001 C CNN
-F 3 "" H 4900 1800 50  0001 C CNN
-	1    4900 1800
+P 5450 1850
+F 0 "#PWR0110" H 5450 1700 50  0001 C CNN
+F 1 "+5V" H 5465 2023 50  0000 C CNN
+F 2 "" H 5450 1850 50  0001 C CNN
+F 3 "" H 5450 1850 50  0001 C CNN
+	1    5450 1850
 	1    0    0    -1
 $EndComp
@@
 	1    0    0    -1
 $EndComp
-$Comp
-L power:+5V #PWR0115
-U 1 1 5B29A63D
-P 7600 2050
-F 0 "#PWR0115" H 7600 1900 50  0001 C CNN
-F 1 "+5V" H 7615 2223 50  0000 C CNN
-F 2 "" H 7600 2050 50  0001 C CNN
-F 3 "" H 7600 2050 50  0001 C CNN
-	1    7600 2050
-	1    0    0    -1
-$EndComp
 Wire Wire Line
 	7700 2200 7600 2200
@@
 L power:GND #PWR0116
 U 1 1 5B29CE6A
-P 8150 3750
-F 0 "#PWR0116" H 8150 3500 50  0001 C CNN
-F 1 "GND" H 8155 3577 50  0000 C CNN
-F 2 "" H 8150 3750 50  0001 C CNN
-F 3 "" H 8150 3750 50  0001 C CNN
-	1    8150 3750
+P 8500 3800
+F 0 "#PWR0116" H 8500 3550 50  0001 C CNN
+F 1 "GND" H 8505 3627 50  0000 C CNN
+F 2 "" H 8500 3800 50  0001 C CNN
+F 3 "" H 8500 3800 50  0001 C CNN
+	1    8500 3800
 	1    0    0    -1
 $EndComp
@@
 L power:+5V #PWR0117
 U 1 1 5B29CEAF
-P 8150 3150
-F 0 "#PWR0117" H 8150 3000 50  0001 C CNN
-F 1 "+5V" H 8165 3323 50  0000 C CNN
-F 2 "" H 8150 3150 50  0001 C CNN
-F 3 "" H 8150 3150 50  0001 C CNN
-	1    8150 3150
-	1    0    0    -1
-$EndComp
-Wire Wire Line
-	8400 3300 8400 3250
-Wire Wire Line
-	8400 3250 8150 3250
-Wire Wire Line
-	7850 3250 7850 3300
-Wire Wire Line
-	8150 3150 8150 3250
-Connection ~ 8150 3250
-Wire Wire Line
-	7850 3600 7850 3650
-Wire Wire Line
-	8400 3650 8400 3600
-Wire Wire Line
-	8150 3750 8150 3650
-Connection ~ 8150 3650
-Wire Wire Line
-	8150 3650 8400 3650
+P 8500 3200
+F 0 "#PWR0117" H 8500 3050 50  0001 C CNN
+F 1 "+5V" H 8515 3373 50  0000 C CNN
+F 2 "" H 8500 3200 50  0001 C CNN
+F 3 "" H 8500 3200 50  0001 C CNN
+	1    8500 3200
+	1    0    0    -1
+$EndComp
+Wire Wire Line
+	8750 3350 8750 3300
+Wire Wire Line
+	8750 3300 8500 3300
+Wire Wire Line
+	8200 3300 8200 3350
+Wire Wire Line
+	8500 3200 8500 3300
+Connection ~ 8500 3300
+Wire Wire Line
+	8200 3650 8200 3700
+Wire Wire Line
+	8750 3700 8750 3650
+Wire Wire Line
+	8500 3800 8500 3700
+Connection ~ 8500 3700
+Wire Wire Line
+	8500 3700 8750 3700
 Wire Notes Line
 	6950 4150 9450 4150
@@
 	4350 5850 9450 5850
 Wire Wire Line
-	7850 3250 8150 3250
-Wire Wire Line
-	7850 3650 8150 3650
-$Comp
-L Device:D D?
+	8200 3300 8500 3300
+Wire Wire Line
+	8200 3700 8500 3700
+$Comp
+L Device:D D9
 U 1 1 5B2AEBA3
-P 5200 1900
-F 0 "D?" H 5200 1684 50  0000 C CNN
-F 1 "1N4007" H 5200 1775 50  0000 C CNN
-F 2 "" H 5200 1900 50  0001 C CNN
-F 3 "~" H 5200 1900 50  0001 C CNN
-	1    5200 1900
+P 7900 3300
+F 0 "D9" H 7900 3084 50  0000 C CNN
+F 1 "1N4007" H 7900 3175 50  0000 C CNN
+F 2 "Diodes_THT:D_DO-41_SOD81_P2.54mm_Vertical_AnodeUp" H 7900 3300 50  0001 C CNN
+F 3 "~" H 7900 3300 50  0001 C CNN
+	1    7900 3300
 	-1   0    0    1
 $EndComp
 Wire Wire Line
-	5350 1900 5450 1900
-Wire Wire Line
-	5450 1900 5450 2150
-Wire Wire Line
-	5050 1900 4900 1900
-Wire Wire Line
-	4900 1900 4900 1800
+	5450 1850 5450 2150
+$Comp
+L power:VCC #PWR0102
+U 1 1 5B2AA17D
+P 7600 2050
+F 0 "#PWR0102" H 7600 1900 50  0001 C CNN
+F 1 "VCC" H 7617 2223 50  0000 C CNN
+F 2 "" H 7600 2050 50  0001 C CNN
+F 3 "" H 7600 2050 50  0001 C CNN
+	1    7600 2050
+	1    0    0    -1
+$EndComp
+$Comp
+L power:VCC #PWR0115
+U 1 1 5B2AA1A9
+P 8600 2050
+F 0 "#PWR0115" H 8600 1900 50  0001 C CNN
+F 1 "VCC" H 8617 2223 50  0000 C CNN
+F 2 "" H 8600 2050 50  0001 C CNN
+F 3 "" H 8600 2050 50  0001 C CNN
+	1    8600 2050
+	1    0    0    -1
+$EndComp
+$Comp
+L power:VCC #PWR0118
+U 1 1 5B2AA1CE
+P 7550 3200
+F 0 "#PWR0118" H 7550 3050 50  0001 C CNN
+F 1 "VCC" H 7567 3373 50  0000 C CNN
+F 2 "" H 7550 3200 50  0001 C CNN
+F 3 "" H 7550 3200 50  0001 C CNN
+	1    7550 3200
+	1    0    0    -1
+$EndComp
+Wire Wire Line
+	7750 3300 7550 3300
+Wire Wire Line
+	7550 3300 7550 3200
+Wire Wire Line
+	8050 3300 8200 3300
+Connection ~ 8200 3300
 $EndSCHEMATC
