File: irblock.sch (KiCad schematic (older format))
At the start: 4 parts, among them Q1 DETECT_0

Commit message: Started PCB layout
Parts:
- removed Q1: DETECT_0, LEDs:LED_D5.0mm, symbol Device:Q_Photo_NPN
- added Q3: DETECT, LEDs:LED_D5.0mm, symbol Device:Q_Photo_NPN_EC
Changed lines of the file:
@@
 $Descr User 5906 5906
 encoding utf-8
-Sheet 2 9
+Sheet 4 9
 Title ""
 Date ""
@@
 Wire Wire Line
 	2750 3000 2750 3150
-$Comp
-L Device:Q_Photo_NPN Q1
-U 1 1 5B320903
-P 3150 2850
-AR Path="/5B31F56C/5B320903" Ref="Q1"  Part="1"
-AR Path="/5B32527D/5B320903" Ref="Q2"  Part="1"
-AR Path="/5B3280EC/5B320903" Ref="Q3"  Part="1"
-AR Path="/5B3280EF/5B320903" Ref="Q4"  Part="1"
-AR Path="/5B32922D/5B320903" Ref="Q5"  Part="1"
-AR Path="/5B329230/5B320903" Ref="Q6"  Part="1"
-AR Path="/5B329235/5B320903" Ref="Q7"  Part="1"
-AR Path="/5B329238/5B320903" Ref="Q8"  Part="1"
-F 0 "Q1" H 3340 2896 50  0000 L CNN
-F 1 "DETECT_0" H 3340 2805 50  0000 L CNN
-F 2 "LEDs:LED_D5.0mm" H 3350 2950 50  0001 C CNN
-F 3 "~" H 3150 2850 50  0001 C CNN
-	1    3150 2850
-	1    0    0    -1
-$EndComp
 Wire Wire Line
 	3250 3050 3250 3150
@@
 Text HLabel 3500 2600 2    50   Output ~ 0
 OUTPUT
+$Comp
+L Device:Q_Photo_NPN_EC Q3
+U 1 1 5B29B338
+P 3350 2850
+AR Path="/5B3280EC/5B29B338" Ref="Q3"  Part="1"
+AR Path="/5B31F56C/5B29B338" Ref="Q1"  Part="1"
+AR Path="/5B32527D/5B29B338" Ref="Q2"  Part="1"
+AR Path="/5B3280EF/5B29B338" Ref="Q4"  Part="1"
+AR Path="/5B32922D/5B29B338" Ref="Q5"  Part="1"
+AR Path="/5B329230/5B29B338" Ref="Q6"  Part="1"
+AR Path="/5B329235/5B29B338" Ref="Q7"  Part="1"
+AR Path="/5B329238/5B29B338" Ref="Q8"  Part="1"
+F 0 "Q1" H 3172 2896 50  0000 R CNN
+F 1 "DETECT" H 3172 2805 50  0000 R CNN
+F 2 "LEDs:LED_D5.0mm" H 3550 2950 50  0001 C CNN
+F 3 "~" H 3350 2850 50  0001 C CNN
+	1    3350 2850
+	-1   0    0    -1
+$EndComp
 $EndSCHEMATC

Commit message: Added library for sensor
Parts:
- Q3: value DETECT -> QSD124
Changed lines of the file:
@@
 AR Path="/5B329235/5B323CD0" Ref="#PWR0130"  Part="1"
 AR Path="/5B329238/5B323CD0" Ref="#PWR0132"  Part="1"
-F 0 "#PWR0132" H 3000 1900 50  0001 C CNN
+F 0 "#PWR0118" H 3000 1900 50  0001 C CNN
 F 1 "+5V" H 3015 2223 50  0000 C CNN
 F 2 "" H 3000 2050 50  0001 C CNN
@@
 AR Path="/5B329235/5B323F60" Ref="#PWR0131"  Part="1"
 AR Path="/5B329238/5B323F60" Ref="#PWR0133"  Part="1"
-F 0 "#PWR0133" H 3000 3000 50  0001 C CNN
+F 0 "#PWR0119" H 3000 3000 50  0001 C CNN
 F 1 "GND" H 3005 3077 50  0000 C CNN
 F 2 "" H 3000 3250 50  0001 C CNN
@@
 AR Path="/5B329238/5B29B338" Ref="Q8"  Part="1"
 F 0 "Q1" H 3172 2896 50  0000 R CNN
-F 1 "DETECT" H 3172 2805 50  0000 R CNN
+F 1 "QSD124" H 3172 2805 50  0000 R CNN
 F 2 "LEDs:LED_D5.0mm" H 3550 2950 50  0001 C CNN
 F 3 "~" H 3350 2850 50  0001 C CNN

Commit message: Added reverse voltage diode
Parts:
- D1: value EMITTER -> HSDL-4420
Connections:
- net labels added: VCC
- net labels removed: +5V
Changed lines of the file:
@@
 AR Path="/5B329238/5B3208F2" Ref="D8"  Part="1"
 F 0 "D1" V 2800 2950 50  0000 L CNN
-F 1 "EMITTER" V 2700 2950 50  0000 L CNN
+F 1 "HSDL-4420" V 2700 2950 50  0000 L CNN
 F 2 "LEDs:LED_D5.0mm" H 2750 2850 50  0001 C CNN
 F 3 "~" H 2750 2850 50  0001 C CNN
@@
 Wire Wire Line
 	3250 2150 3000 2150
-$Comp
-L power:+5V #PWR0118
-U 1 1 5B323CD0
-P 3000 2050
-AR Path="/5B31F56C/5B323CD0" Ref="#PWR0118"  Part="1"
-AR Path="/5B32527D/5B323CD0" Ref="#PWR0120"  Part="1"
-AR Path="/5B3280EC/5B323CD0" Ref="#PWR0122"  Part="1"
-AR Path="/5B3280EF/5B323CD0" Ref="#PWR0124"  Part="1"
-AR Path="/5B32922D/5B323CD0" Ref="#PWR0126"  Part="1"
-AR Path="/5B329230/5B323CD0" Ref="#PWR0128"  Part="1"
-AR Path="/5B329235/5B323CD0" Ref="#PWR0130"  Part="1"
-AR Path="/5B329238/5B323CD0" Ref="#PWR0132"  Part="1"
-F 0 "#PWR0118" H 3000 1900 50  0001 C CNN
-F 1 "+5V" H 3015 2223 50  0000 C CNN
-F 2 "" H 3000 2050 50  0001 C CNN
-F 3 "" H 3000 2050 50  0001 C CNN
-	1    3000 2050
-	1    0    0    -1
-$EndComp
 Wire Wire Line
 	3000 2150 3000 2050
@@
 	-1   0    0    -1
 $EndComp
+$Comp
+L power:VCC #PWR?
+U 1 1 5B2AF7C6
+P 3000 2050
+F 0 "#PWR?" H 3000 1900 50  0001 C CNN
+F 1 "VCC" H 3017 2223 50  0000 C CNN
+F 2 "" H 3000 2050 50  0001 C CNN
+F 3 "" H 3000 2050 50  0001 C CNN
+	1    3000 2050
+	1    0    0    -1
+$EndComp
 $EndSCHEMATC
